File: Celestron-Ethernet.kicad_pcb (KiCad board)
At the start: 4 copper layers, 88.9 x 31.8 mm, 69 parts, among them J1 Joystick, J2 GPS, J3 6P6C, J4 RJ45_Amphenol_RJMG1BD3B8K1ANR, SW1 SW_DIP_x02, SW2 SW_Push, U1 74AHC1G125, U2 ATmega328P-AU, U3 NCV33375ST-3.3, U4 W5500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

Commit message: finished routing
Parts:
- moved C6 41.5 mm to (170.2, 100.5)
- moved C7 14.0 mm to (156.2, 100.3)
- moved R20 10.2 mm to (134.6, 109.0)
- moved U1 7.80 mm to (141.0, 109.2)
- moved C5 7.62 mm to (147.3, 104.8)
- moved C16 5.08 mm to (121.9, 109.0)
- moved R21 5.08 mm to (127.0, 109.0)
- moved R9 4.90 mm to (124.5, 87.9)
- moved C2 4.32 mm to (151.1, 104.8), turned to 90 degrees
- moved Y1 4.32 mm to (154.9, 106.7)
- moved C3 4.19 mm to (151.1, 109.0)
- moved C17 4.19 mm to (121.9, 92.1), turned to 90 degrees
- moved C19 2.54 mm to (129.5, 109.0)
- moved C25 2.54 mm to (139.7, 104.8)
- moved C12 2.54 mm to (124.5, 104.8)
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Routing:
- net VCC: track 0.00 -> 123.7 mm, vias 0 -> 21
- net GND: track 0.00 -> 70.9 mm, vias 0 -> 34
- net /SCK: track 0.00 -> 61.8 mm, vias 0 -> 3
- net /GRX: track 0.00 -> 49.0 mm, vias 0 -> 2
- net /GTX: track 0.00 -> 47.3 mm, vias 0 -> 2
- net /W5500/LEDY_K: track 0.00 -> 38.6 mm
- net /MOSI: track 0.00 -> 37.9 mm, vias 0 -> 2
- net /MISO: track 0.00 -> 37.0 mm, vias 0 -> 2
- net /~RST: track 0.00 -> 35.8 mm, vias 0 -> 2
- net /TXO: track 0.00 -> 30.5 mm, vias 0 -> 2
- net /W5500/LEDG_K: track 0.00 -> 29.2 mm
- net +3.3VA: track 0.00 -> 23.9 mm, vias 0 -> 10
- net /W5500/TD-: track 0.00 -> 22.4 mm
- net /BUSY: track 0.00 -> 22.1 mm, vias 0 -> 2
- net GNDPWR: track 0.00 -> 21.2 mm
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Other:
- net class Default: trace_width 0.1524 -> 0.2032
- rule pad_to_mask_clearance: 0.0508 -> 0
- rule trace_min: 0.1524 -> 0.2032
- board text removed: "DCHP Client"
- board text removed: "EVO WiFi ON"

Commit message: final version
Parts:
- removed C27: 100nF, Capacitor_SMD:C_0603_1608Metric
- removed the C5 at (147.3, 104.8)
- removed the C6 at (170.2, 100.5)
- removed the R1 at (144.8, 104.8)
- removed the U1 at (141.0, 109.2)
- added C11: 6.8nF, Capacitor_SMD:C_0603_1608Metric, F.Cu at (125.7, 104.8)
- added C7: 100nF, Capacitor_SMD:C_0603_1608Metric, F.Cu at (170.2, 100.3)
- added R2: 330R, Resistor_SMD:R_0603_1608Metric, F.Cu at (146.1, 104.8)
- added U2: 74AHC1G125, Package_TO_SOT_SMD:SOT-23-5, F.Cu at (142.2, 109.2)
- C10: renamed from C11; value 1uF -> 100nF
- C13: value 6.8nF -> 18pF
- C15: value 18pF -> 10nF
- C16: value 10nF -> 22nF
- C17: value 22nF -> 1nF/2KV; footprint Capacitor_SMD:C_0603_1608Metric -> Capacitor_SMD:C_1206_3216Metric
- C18: value 1nF/2KV -> 4.7uF; footprint Capacitor_SMD:C_1206_3216Metric -> Capacitor_SMD:C_0603_1608Metric
- C19: value 4.7uF -> 10nF
- C20: value 10nF -> 100nF
- C21: value 100nF -> 1uF
- C22: value 1uF -> 10uF
- C23, C25: value 10uF -> 100nF
- C24: value 100nF -> 10uF
- moved C15 27.3 mm to (123.2, 109.0)
- moved R5 26.4 mm to (149.9, 87.9)
- moved D3 26.4 mm to (149.9, 92.1)
- moved C13 24.1 mm to (148.6, 100.5)
- moved C9 22.9 mm to (172.7, 109.0), turned to 270 degrees
- moved C17 19.7 mm to (117.6, 111.3)
- moved C23 19.5 mm to (141.0, 100.5)
- moved C25 17.8 mm to (134.1, 87.9)
- moved C16 16.9 mm to (123.2, 92.1)
- moved R4 15.4 mm to (161.3, 90.2)
- moved C18 14.7 mm to (130.8, 109.0)
- moved C20 13.3 mm to (128.3, 96.3)
- moved C26 8.13 mm to (141.0, 87.9)
- moved C12 4.50 mm to (125.7, 100.5)
- moved C24 4.50 mm to (141.0, 104.8), turned to 270 degrees
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- renumbered C7 to C5, C8 to C6, C10 to C8, R2 to R1, U2 to U1
Connections:
- C12 pad 1: /W5500/RX+ -> /W5500/RD-
- C12 pad 2: /W5500/RD+ -> /W5500/RX-
- C13 pad 1: /W5500/RD- -> GND
- C13 pad 2: /W5500/RX- -> Net-(C13-Pad2)
- C15 pad 2: Net-(C15-Pad2) -> /W5500/RCT
- C16 pad 2: /W5500/RCT -> /W5500/TCT
- C17 pad 2: /W5500/TCT -> GNDPWR
- C18 pad 2: GNDPWR -> Net-(C18-Pad2)
- C20 pad 1: GND -> +3.3VA
- C20 pad 2: Net-(C20-Pad2) -> GND
- C23 pad 1: +3.3VA -> VCC
- C25 pad 1: VCC -> +3.3VA
- C26 pad 1: +3.3VA -> VCC
- J4 pad R7: Net-(J4-PadR7) -> (no net)
- R18 pad 1: Net-(C15-Pad2) -> Net-(C14-Pad2)
- R18 pad 2: Net-(C14-Pad2) -> Net-(C13-Pad2)
- U1 pad 1: Net-(U2-Pad1) -> (no net)
- U1 pad 13: Net-(U2-Pad13) -> (no net)
- U1 pad 14: Net-(U2-Pad14) -> (no net)
- U1 pad 19: Net-(U2-Pad19) -> (no net)
- U1 pad 22: Net-(U2-Pad22) -> (no net)
- U1 pad 24: Net-(U2-Pad24) -> (no net)
- U1 pad 25: Net-(U2-Pad25) -> (no net)
- U1 pad 32: Net-(U2-Pad32) -> (no net)
- U4 pad 12: Net-(U4-Pad12) -> (no net)
- U4 pad 13: Net-(U4-Pad13) -> (no net)
- U4 pad 18: Net-(U4-Pad18) -> (no net)
- U4 pad 20: Net-(C19-Pad2) -> Net-(C18-Pad2)
- U4 pad 22: Net-(C20-Pad2) -> Net-(C19-Pad2)
- U4 pad 24: Net-(U4-Pad24) -> (no net)
- U4 pad 26: Net-(U4-Pad26) -> (no net)
- U4 pad 30: Net-(C14-Pad2) -> Net-(C13-Pad2)
- U4 pad 31: Net-(C15-Pad2) -> Net-(C14-Pad2)
- U4 pad 46: Net-(U4-Pad46) -> (no net)
- U4 pad 47: Net-(U4-Pad47) -> (no net)
- U4 pad 7: Net-(U4-Pad7) -> (no net)
- Y2 pad 1: Net-(C15-Pad2) -> Net-(C14-Pad2)
- Y2 pad 2: Net-(C14-Pad2) -> Net-(C13-Pad2)
Routing:
- net Net-(C13-Pad2): track 0.00 -> 12.4 mm
- net Net-(C15-Pad2): track 12.1 -> 0.00 mm
- net Net-(C18-Pad2): track 0.00 -> 7.62 mm
- net Net-(C20-Pad2): track 7.26 -> 0.00 mm
- net /GRX: track 49.0 -> 53.0 mm
- net /GTX: track 47.3 -> 50.1 mm
- net /TXO: track 30.5 -> 28.4 mm, vias 2 -> 1
- net /DTR: track 21.0 -> 22.6 mm
- net /TX: track 2.94 -> 4.32 mm
- net /MISO: track 37.0 -> 35.7 mm
- net /MOSI: track 37.9 -> 36.7 mm
- net /~RST: track 35.8 -> 34.6 mm
- net /SCK: track 61.8 -> 62.7 mm
- net GND: track 70.9 -> 71.8 mm, vias 34 -> 63
- net /~RESET: track 19.7 -> 19.1 mm, vias 3 -> 2
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Other:
- board text added: "Celestron Ethernet Adapter v1.0 by Hyiger Designs"
- board text removed: "Celestron Ethernet Adapter v 1.0 by Hyiger Designs"
- board text removed: "On - DCHP Client Off - DHCP Server"

Commit message: sent to fab
Parts:
- moved FB1 0.76 mm to (137.5, 87.1)
Routing:
- net GND: track 71.8 -> 78.3 mm, vias 63 -> 66
- net /SCK: track 62.7 -> 61.4 mm
- net VCC: track 123.4 -> 122.7 mm
