File: Programming-Adapter/Programming-Adapter.kicad_pcb (KiCad board)
At the start: 2 copper layers, 25.4 x 16.3 mm, 2 parts, among them J1 FTDI, J2 6P6C

Commit message: update
Routing:
- net /DTR: track 22.9 -> 25.5 mm
- net GND: vias 9 -> 0
Other:
- board text added: "Programming Adapter v1.0 Hyiger Designs"
Changed lines of the file:
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@@
   (general
     (thickness 1.6)
-    (drawings 9)
-    (tracks 22)
+    (drawings 10)
+    (tracks 14)
     (zones 0)
     (modules 2)
@@
   (page A4)
   (layers
-    (0 F.Cu signal)
+    (0 F.Cu signal hide)
     (31 B.Cu signal)
     (36 B.SilkS user)
@@
     (45 Margin user)
     (46 B.CrtYd user)
-    (47 F.CrtYd user)
+    (47 F.CrtYd user hide)
   )
   (setup
@@
     (user_trace_width 0.4064)
     (trace_clearance 0.2)
-    (zone_clearance 0.508)
+    (zone_clearance 0.254)
     (zone_45_only no)
     (trace_min 0.2)
@@
     )
   )
-  (gr_text GND (at 167.386 84.328) (layer F.SilkS)
-    (effects (font (size 0.8128 0.8128) (thickness 0.1524)))
-  )
-  (gr_text VCC (at 167.308591 79.248) (layer F.SilkS)
-    (effects (font (size 0.8128 0.8128) (thickness 0.1524)))
-  )
-  (gr_text RXI (at 167.134419 76.708) (layer F.SilkS)
-    (effects (font (size 0.8128 0.8128) (thickness 0.1524)))
-  )
-  (gr_text TXO (at 167.269886 74.041) (layer F.SilkS)
-    (effects (font (size 0.8128 0.8128) (thickness 0.1524)))
-  )
-  (gr_text DTR (at 167.269886 71.501) (layer F.SilkS)
+  (gr_text "Programming\nAdapter v1.0\nHyiger Designs" (at 179.07 77.978) (layer B.SilkS)
+    (effects (font (size 0.8128 0.8128) (thickness 0.1524)) (justify mirror))
+  )
+  (gr_text GND (at 167.64 84.201) (layer F.SilkS)
+    (effects (font (size 0.8128 0.8128) (thickness 0.1524)))
+  )
+  (gr_text VCC (at 167.562591 79.121) (layer F.SilkS)
+    (effects (font (size 0.8128 0.8128) (thickness 0.1524)))
+  )
+  (gr_text RXI (at 167.388419 76.581) (layer F.SilkS)
+    (effects (font (size 0.8128 0.8128) (thickness 0.1524)))
+  )
+  (gr_text TXO (at 167.523886 74.041) (layer F.SilkS)
+    (effects (font (size 0.8128 0.8128) (thickness 0.1524)))
+  )
+  (gr_text DTR (at 167.523886 71.501) (layer F.SilkS)
     (effects (font (size 0.8128 0.8128) (thickness 0.1524)))
   )
@@
   (gr_line (start 186.309 69.723) (end 186.309 85.979) (layer Edge.Cuts) (width 0.05))
   (gr_line (start 160.909 69.723) (end 186.309 69.723) (layer Edge.Cuts) (width 0.05))
-  (segment (start 173.99 81.026) (end 170.434 81.026) (width 0.4064) (layer B.Cu) (net 1) (status 20))
-  (segment (start 175.006 80.01) (end 173.99 81.026) (width 0.4064) (layer B.Cu) (net 1))
-  (segment (start 175.006 72.644) (end 175.006 80.01) (width 0.4064) (layer B.Cu) (net 1))
-  (segment (start 173.868 71.506) (end 175.006 72.644) (width 0.4064) (layer B.Cu) (net 1))
+  (segment (start 171.958 82.55) (end 170.434 81.026) (width 0.4064) (layer B.Cu) (net 1) (status 20))
+  (segment (start 174.244 82.55) (end 171.958 82.55) (width 0.4064) (layer B.Cu) (net 1))
+  (segment (start 175.387 81.407) (end 174.244 82.55) (width 0.4064) (layer B.Cu) (net 1))
+  (segment (start 175.387 73.025) (end 175.387 81.407) (width 0.4064) (layer B.Cu) (net 1))
+  (segment (start 173.868 71.506) (end 175.387 73.025) (width 0.4064) (layer B.Cu) (net 1))
   (segment (start 164.973 71.506) (end 173.868 71.506) (width 0.4064) (layer B.Cu) (net 1) (status 10))
   (segment (start 172.974 76.581) (end 172.974 77.216) (width 0.4064) (layer F.Cu) (net 2) (status 30))
@@
   (segment (start 169.794 79.126) (end 170.434 78.486) (width 0.4064) (layer B.Cu) (net 4) (status 20))
   (segment (start 164.973 79.126) (end 169.794 79.126) (width 0.4064) (layer B.Cu) (net 4) (status 10))
-  (via (at 167.767 78.232) (size 0.8128) (drill 0.4064) (layers F.Cu B.Cu) (net 5))
-  (via (at 167.767 81.407) (size 0.8128) (drill 0.4064) (layers F.Cu B.Cu) (net 5))
-  (via (at 167.767 84.582) (size 0.8128) (drill 0.4064) (layers F.Cu B.Cu) (net 5))
-  (via (at 162.433 78.232) (size 0.8128) (drill 0.4064) (layers F.Cu B.Cu) (net 5))
-  (via (at 162.433 81.407) (size 0.8128) (drill 0.4064) (layers F.Cu B.Cu) (net 5))
-  (via (at 162.433 84.582) (size 0.8128) (drill 0.4064) (layers F.Cu B.Cu) (net 5))
-  (via (at 162.433 71.882) (size 0.8128) (drill 0.4064) (layers F.Cu B.Cu) (net 5))
-  (via (at 167.767 75.057) (size 0.8128) (drill 0.4064) (layers F.Cu B.Cu) (net 5))
-  (via (at 162.433 75.057) (size 0.8128) (drill 0.4064) (layers F.Cu B.Cu) (net 5))
   (zone (net 5) (net_name GND) (layer B.Cu) (hatch edge 0.508)
-    (connect_pads (clearance 0.508))
+    (connect_pads (clearance 0.254))
     (min_thickness 0.254)
-    (fill yes (arc_segments 32) (thermal_gap 0.254) (thermal_bridge_width 0.4064))
+    (fill (arc_segments 32) (thermal_gap 0.254) (thermal_bridge_width 0.4064))
     (polygon
       (pts
-        (xy 187.706 85.979) (xy 160.909 85.979) (xy 160.909 69.723) (xy 187.706 69.723)
+        (xy 186.309 85.979) (xy 160.909 85.979) (xy 160.909 69.723) (xy 186.309 69.723)
       )
     )
@@
     (connect_pads (clearance 0.254))
     (min_thickness 0.254)
-    (fill yes (arc_segments 32) (thermal_gap 0.254) (thermal_bridge_width 0.4064))
+    (fill (arc_segments 32) (thermal_gap 0.254) (thermal_bridge_width 0.4064))
     (polygon
       (pts
-        (xy 187.706 85.979) (xy 160.909 85.979) (xy 160.909 69.723) (xy 187.706 69.723)
+        (xy 186.309 85.979) (xy 160.909 85.979) (xy 160.909 69.723) (xy 186.309 69.723)
       )
     )
