File: Joystick/Joystick.sch (KiCad schematic (older format))
At the start: 11 parts, among them J1 Joystick, SW1 Plus, SW2 Minus, SW3 Down, SW4 Up, SW5 Right, SW6 Left, SW7 Center, U1 HDSP-A153, U2 AS1115-BSST

Commit message: keypad
Parts:
- added H1, H2, H3, H4: *, MountingHole:MountingHole_3.2mm_M3_Pad_Via, symbol Mechanical:MountingHole_Pad
Connections:
- net GND: now also H1.1, H2.1, H3.1, H4.1
- net at U1.10 (A), U2.15 (SEGA): now also SW5.1 (A); no longer SW1.2 (B)
- net at U1.2 (F), U2.16 (SEGF): now also SW3.1 (A); no longer SW4.1 (A)
- net at U1.3 (G), U2.18 (SEGG): now also SW4.1 (A); no longer SW2.1 (A)
- net at U1.4 (E), U2.21 (SEGE): now also SW2.1 (A); no longer SW6.1 (A)
- net at U1.5 (D), U2.23 (SEGD): now also SW1.1 (A); no longer SW7.2 (B)
- net at U1.8 (C), U2.20 (SEGC): now also SW7.1 (A); no longer SW5.2 (B)
- net at U1.9 (B), U2.17 (SEGB): now also SW6.1 (A); no longer SW3.2 (B)
- net at SW2.2 (B), SW4.2 (B), SW6.2 (B)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: now also SW1.2 (B), SW3.2 (B), SW5.2 (B), SW7.2 (B); no longer SW1.1 (A), SW3.1 (A), SW5.1 (A), SW7.1 (A)
Other:
- moved on the sheet: SW1, SW2, SW3, SW4, SW5, SW6, SW7
